File: elen433_honors_solar_cell_project.kicad_sch (KiCad schematic)
At the start: 6 parts, among them J1 Conn_01x02

Commit message: Created board
Connections:
- net +5V: now also U1.1 (pos); no longer U1. (pos2)
- net GND: now also U1.2 (neg); no longer U1. (pos2)
Changed lines of the file:
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@@
 	(generator_version "8.0")
 	(paper "A4")
-	(junction
-		(at 101.6 63.5)
-		(diameter 0)
-		(color 0 0 0 0)
-	)
-	(junction
-		(at 78.74 53.34)
-		(diameter 0)
-		(color 0 0 0 0)
-	)
 	(wire
 		(pts
@@
 	(wire
 		(pts
-			(xy 78.74 63.5) (xy 81.28 63.5)
-		)
-		(stroke
-			(width 0)
-			(type default)
-		)
-	)
-	(wire
-		(pts
 			(xy 133.35 63.5) (xy 133.35 66.04)
 		)
@@
 	(wire
 		(pts
-			(xy 78.74 53.34) (xy 78.74 63.5)
-		)
-		(stroke
-			(width 0)
-			(type default)
-		)
-	)
-	(wire
-		(pts
 			(xy 109.22 43.18) (xy 113.03 43.18)
 		)
@@
 	(wire
 		(pts
-			(xy 99.06 53.34) (xy 101.6 53.34)
-		)
-		(stroke
-			(width 0)
-			(type default)
-		)
-	)
-	(wire
-		(pts
-			(xy 101.6 63.5) (xy 101.6 66.04)
-		)
-		(stroke
-			(width 0)
-			(type default)
-		)
-	)
-	(wire
-		(pts
 			(xy 109.22 45.72) (xy 109.22 48.26)
 		)
@@
 	(wire
 		(pts
-			(xy 101.6 53.34) (xy 101.6 63.5)
-		)
-		(stroke
-			(width 0)
-			(type default)
-		)
-	)
-	(wire
-		(pts
-			(xy 99.06 63.5) (xy 101.6 63.5)
+			(xy 101.6 59.69) (xy 101.6 66.04)
 		)
 		(stroke
@@
 	(wire
 		(pts
-			(xy 78.74 53.34) (xy 81.28 53.34)
-		)
-		(stroke
-			(width 0)
-			(type default)
-		)
-	)
-	(wire
-		(pts
-			(xy 78.74 50.8) (xy 78.74 53.34)
+			(xy 78.74 59.69) (xy 81.28 59.69)
+		)
+		(stroke
+			(width 0)
+			(type default)
+		)
+	)
+	(wire
+		(pts
+			(xy 99.06 59.69) (xy 101.6 59.69)
+		)
+		(stroke
+			(width 0)
+			(type default)
+		)
+	)
+	(wire
+		(pts
+			(xy 78.74 53.34) (xy 78.74 59.69)
 		)
 		(stroke
@@
 	(symbol
 		(lib_id "solar:solar_cell")
-		(at 90.17 58.42 0)
+		(at 90.17 64.77 0)
 		(unit 1)
 		(exclude_from_sim no)
@@
 		(fields_autoplaced yes)
 		(property "Reference" "U1"
-			(at 90.17 49.53 0)
+			(at 90.17 55.88 0)
 			(effects
 				(font
@@
 		)
 		(property "Value" "~"
-			(at 90.17 52.07 0)
+			(at 90.17 58.42 0)
 			(effects
 				(font
@@
 		)
 		(property "Footprint" "solar:Solar"
-			(at 88.9 58.42 0)
+			(at 88.9 64.77 0)
 			(effects
 				(font
@@
 		)
 		(property "Datasheet" ""
-			(at 88.9 58.42 0)
+			(at 88.9 64.77 0)
 			(effects
 				(font
@@
 		)
 		(property "Description" "Solar Cell"
-			(at 90.17 59.69 0)
-			(effects
-				(font
-					(size 1.27 1.27)
-				)
-				(hide yes)
-			)
-		)
-		(pin ""
-		)
-		(pin ""
-		)
-		(pin ""
-		)
-		(pin ""
+			(at 90.17 66.04 0)
+			(effects
+				(font
+					(size 1.27 1.27)
+				)
+				(hide yes)
+			)
+		)
+		(pin "1"
+		)
+		(pin "2"
 		)
 		(instances
@@
 	(symbol
 		(lib_id "power:+5V")
-		(at 78.74 50.8 0)
+		(at 78.74 53.34 0)
 		(unit 1)
 		(exclude_from_sim no)
@@
 		(fields_autoplaced yes)
 		(property "Reference" "#PWR01"
-			(at 78.74 54.61 0)
+			(at 78.74 57.15 0)
 			(effects
 				(font
@@
 		)
 		(property "Value" "+5V"
-			(at 78.74 45.72 0)
+			(at 78.74 48.26 0)
 			(effects
 				(font
@@
 		)
 		(property "Footprint" ""
-			(at 78.74 50.8 0)
+			(at 78.74 53.34 0)
 			(effects
 				(font
@@
 		)
 		(property "Datasheet" ""
-			(at 78.74 50.8 0)
+			(at 78.74 53.34 0)
 			(effects
 				(font
@@
 		)
 		(property "Description" "Power symbol creates a global label with name \"+5V\""
-			(at 78.74 50.8 0)
-			(effects
-				(font
+			(at 78.74 53.34 0)
+			(effects
+				(font
